File: PCB_POWER_DISTRIBUTION/RACK_CONNECTOR_V2/RACK_CONNECTOR_V2/RACK_CONNECTOR_V2/RACK_CONNECTOR_V2.kicad_sch (KiCad schematic)
At the start: 24 parts, among them J1 A-DS_09_A_KG-T2S, J10 Conn_01x09_Female, J11 Conn_01x09_Female, J12 Conn_01x09_Female, J13 A-DS_09_A_KG-T2S, J14 A-DS_09_A_KG-T2S, J15 A-DS_09_A_KG-T2S, J16 A-DS_09_A_KG-T2S, J17 XT90PW-F, J18 XT90PW-F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

Commit message: all the footprint and rooting is done
Parts:
- added J25, J26, J27, J28: Conn_01x09_Female, Connector_PinHeader_2.54mm:PinHeader_1x09_P2.54mm_Vertical, symbol Connector:Conn_01x09_Female
Connections:
- net at J12.9 (Pin_9), J16.1: now also J28.9 (Pin_9)
- net at J12.8 (Pin_8), J16.2: now also J28.8 (Pin_8)
- net at J12.7 (Pin_7), J16.3: now also J28.7 (Pin_7)
- net at J12.6 (Pin_6), J16.4: now also J28.6 (Pin_6)
- net at J12.5 (Pin_5), J16.5: now also J28.5 (Pin_5)
- net at J12.4 (Pin_4), J16.6: now also J28.4 (Pin_4)
- net at J12.3 (Pin_3), J16.7: now also J28.3 (Pin_3)
- net at J12.2 (Pin_2), J16.8: now also J28.2 (Pin_2)
- net at J12.1 (Pin_1), J16.9: now also J28.1 (Pin_1)
- net at J13.1, J9.9 (Pin_9): now also J25.9 (Pin_9)
- net at J13.2, J9.8 (Pin_8): now also J25.8 (Pin_8)
- net at J13.3, J9.7 (Pin_7): now also J25.7 (Pin_7)
- net at J13.4, J9.6 (Pin_6): now also J25.6 (Pin_6)
- net at J13.5, J9.5 (Pin_5): now also J25.5 (Pin_5)
- net at J13.6, J9.4 (Pin_4): now also J25.4 (Pin_4)
- net at J13.7, J9.3 (Pin_3): now also J25.3 (Pin_3)
- net at J13.8, J9.2 (Pin_2): now also J25.2 (Pin_2)
- net at J13.9, J9.1 (Pin_1): now also J25.1 (Pin_1)
- net at J10.9 (Pin_9), J14.1: now also J26.9 (Pin_9)
- net at J10.8 (Pin_8), J14.2: now also J26.8 (Pin_8)
- net at J10.7 (Pin_7), J14.3: now also J26.7 (Pin_7)
- net at J10.6 (Pin_6), J14.4: now also J26.6 (Pin_6)
- net at J10.5 (Pin_5), J14.5: now also J26.5 (Pin_5)
- net at J10.4 (Pin_4), J14.6: now also J26.4 (Pin_4)
- net at J10.3 (Pin_3), J14.7: now also J26.3 (Pin_3)
- net at J10.2 (Pin_2), J14.8: now also J26.2 (Pin_2)
- net at J10.1 (Pin_1), J14.9: now also J26.1 (Pin_1)
- net at J11.1 (Pin_1), J15.9: now also J27.1 (Pin_1)
- net at J11.2 (Pin_2), J15.8: now also J27.2 (Pin_2)
- net at J11.3 (Pin_3), J15.7: now also J27.3 (Pin_3)
- net at J11.4 (Pin_4), J15.6: now also J27.4 (Pin_4)
- net at J11.5 (Pin_5), J15.5: now also J27.5 (Pin_5)
- net at J11.6 (Pin_6), J15.4: now also J27.6 (Pin_6)
- net at J11.7 (Pin_7), J15.3: now also J27.7 (Pin_7)
- net at J11.8 (Pin_8), J15.2: now also J27.8 (Pin_8)
- net at J11.9 (Pin_9), J15.1: now also J27.9 (Pin_9)
Changed lines of the file:
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@@
 (kicad_sch (version 20211123) (generator eeschema)
   (paper "A4")
+  (junction (at 115.57 152.4) (diameter 0) (color 0 0 0 0)
+  )
+  (junction (at 114.3 115.57) (diameter 0) (color 0 0 0 0)
+  )
+  (junction (at 115.57 154.94) (diameter 0) (color 0 0 0 0)
+  )
+  (junction (at 114.3 44.45) (diameter 0) (color 0 0 0 0)
+  )
+  (junction (at 115.57 144.78) (diameter 0) (color 0 0 0 0)
+  )
+  (junction (at 114.3 102.87) (diameter 0) (color 0 0 0 0)
+  )
+  (junction (at 115.57 149.86) (diameter 0) (color 0 0 0 0)
+  )
+  (junction (at 115.57 137.16) (diameter 0) (color 0 0 0 0)
+  )
+  (junction (at 114.3 105.41) (diameter 0) (color 0 0 0 0)
+  )
+  (junction (at 115.57 142.24) (diameter 0) (color 0 0 0 0)
+  )
+  (junction (at 114.3 100.33) (diameter 0) (color 0 0 0 0)
+  )
+  (junction (at 115.57 139.7) (diameter 0) (color 0 0 0 0)
+  )
+  (junction (at 114.3 34.29) (diameter 0) (color 0 0 0 0)
+  )
+  (junction (at 114.3 74.93) (diameter 0) (color 0 0 0 0)
+  )
+  (junction (at 114.3 118.11) (diameter 0) (color 0 0 0 0)
+  )
+  (junction (at 114.3 36.83) (diameter 0) (color 0 0 0 0)
+  )
+  (junction (at 114.3 107.95) (diameter 0) (color 0 0 0 0)
+  )
+  (junction (at 114.3 110.49) (diameter 0) (color 0 0 0 0)
+  )
+  (junction (at 115.57 147.32) (diameter 0) (color 0 0 0 0)
+  )
+  (junction (at 115.57 157.48) (diameter 0) (color 0 0 0 0)
+  )
+  (junction (at 114.3 80.01) (diameter 0) (color 0 0 0 0)
+  )
+  (junction (at 114.3 120.65) (diameter 0) (color 0 0 0 0)
+  )
+  (junction (at 114.3 72.39) (diameter 0) (color 0 0 0 0)
+  )
+  (junction (at 114.3 41.91) (diameter 0) (color 0 0 0 0)
+  )
+  (junction (at 114.3 67.31) (diameter 0) (color 0 0 0 0)
+  )
+  (junction (at 114.3 77.47) (diameter 0) (color 0 0 0 0)
+  )
+  (junction (at 114.3 69.85) (diameter 0) (color 0 0 0 0)
+  )
+  (junction (at 114.3 85.09) (diameter 0) (color 0 0 0 0)
+  )
+  (junction (at 114.3 39.37) (diameter 0) (color 0 0 0 0)
+  )
+  (junction (at 114.3 82.55) (diameter 0) (color 0 0 0 0)
+  )
+  (junction (at 114.3 31.75) (diameter 0) (color 0 0 0 0)
+  )
+  (junction (at 114.3 29.21) (diameter 0) (color 0 0 0 0)
+  )
+  (junction (at 114.3 113.03) (diameter 0) (color 0 0 0 0)
+  )
+  (junction (at 114.3 46.99) (diameter 0) (color 0 0 0 0)
+  )
+  (junction (at 114.3 64.77) (diameter 0) (color 0 0 0 0)
+  )
+  (junction (at 114.3 49.53) (diameter 0) (color 0 0 0 0)
+  )
   (wire (pts (xy 227.33 62.23) (xy 238.76 62.23))
     (stroke (width 0) (type default) (color 0 0 0 0))
@@
     (pin "P")
   )
+  (symbol (lib_id "Connector:Conn_01x09_Female") (at 119.38 74.93 0) (unit 1)
+    (in_bom yes) (on_board yes) (fields_autoplaced)
+    (property "Reference" "J26" (id 0) (at 120.65 73.6599 0)
+      (effects (font (size 1.27 1.27)) (justify left))
+    )
+    (property "Value" "Conn_01x09_Female" (id 1) (at 120.65 76.1999 0)
+      (effects (font (size 1.27 1.27)) (justify left))
+    )
+    (property "Footprint" "Connector_PinHeader_2.54mm:PinHeader_1x09_P2.54mm_Vertical" (id 2) (at 119.38 74.93 0)
+      (effects (font (size 1.27 1.27)) hide)
+    )
+    (property "Datasheet" "~" (id 3) (at 119.38 74.93 0)
+      (effects (font (size 1.27 1.27)) hide)
+    )
+    (pin "1")
+    (pin "2")
+    (pin "3")
+    (pin "4")
+    (pin "5")
+    (pin "6")
+    (pin "7")
+    (pin "8")
+    (pin "9")
+  )
   (symbol (lib_id "SEB:XT90PW-F") (at 222.25 45.72 0) (unit 1)
     (in_bom yes) (on_board yes) (fields_autoplaced)
@@
     (pin "P")
   )
+  (symbol (lib_id "Connector:Conn_01x09_Female") (at 120.65 147.32 0) (unit 1)
+    (in_bom yes) (on_board yes) (fields_autoplaced)
+    (property "Reference" "J28" (id 0) (at 121.92 146.0499 0)
+      (effects (font (size 1.27 1.27)) (justify left))
+    )
+    (property "Value" "Conn_01x09_Female" (id 1) (at 121.92 148.5899 0)
+      (effects (font (size 1.27 1.27)) (justify left))
+    )
+    (property "Footprint" "Connector_PinHeader_2.54mm:PinHeader_1x09_P2.54mm_Vertical" (id 2) (at 120.65 147.32 0)
+      (effects (font (size 1.27 1.27)) hide)
+    )
+    (property "Datasheet" "~" (id 3) (at 120.65 147.32 0)
+      (effects (font (size 1.27 1.27)) hide)
+    )
+    (pin "1")
+    (pin "2")
+    (pin "3")
+    (pin "4")
+    (pin "5")
+    (pin "6")
+    (pin "7")
+    (pin "8")
+    (pin "9")
+  )
   (symbol (lib_id "SEB:A-DS_09_A_KG-T2S") (at 52.07 157.48 180) (unit 1)
     (in_bom yes) (on_board yes) (fields_autoplaced)
@@
     (pin "P")
   )
+  (symbol (lib_id "Connector:Conn_01x09_Female") (at 119.38 110.49 0) (unit 1)
+    (in_bom yes) (on_board yes) (fields_autoplaced)
+    (property "Reference" "J27" (id 0) (at 120.65 109.2199 0)
+      (effects (font (size 1.27 1.27)) (justify left))
+    )
+    (property "Value" "Conn_01x09_Female" (id 1) (at 120.65 111.7599 0)
+      (effects (font (size 1.27 1.27)) (justify left))
+    )
+    (property "Footprint" "Connector_PinHeader_2.54mm:PinHeader_1x09_P2.54mm_Vertical" (id 2) (at 119.38 110.49 0)
+      (effects (font (size 1.27 1.27)) hide)
+    )
+    (property "Datasheet" "~" (id 3) (at 119.38 110.49 0)
+      (effects (font (size 1.27 1.27)) hide)
+    )
+    (pin "1")
+    (pin "2")
+    (pin "3")
+    (pin "4")
+    (pin "5")
+    (pin "6")
+    (pin "7")
+    (pin "8")
+    (pin "9")
+  )
   (symbol (lib_id "SEB:A-DS_09_A_KG-T2S") (at 50.8 120.65 180) (unit 1)
     (in_bom yes) (on_board yes) (fields_autoplaced)
@@
     (pin "P")
   )
+  (symbol (lib_id "Connector:Conn_01x09_Female") (at 119.38 39.37 0) (unit 1)
+    (in_bom yes) (on_board yes) (fields_autoplaced)
+    (property "Reference" "J25" (id 0) (at 120.65 38.0999 0)
+      (effects (font (size 1.27 1.27)) (justify left))
+    )
+    (property "Value" "Conn_01x09_Female" (id 1) (at 120.65 40.6399 0)
+      (effects (font (size 1.27 1.27)) (justify left))
+    )
+    (property "Footprint" "Connector_PinHeader_2.54mm:PinHeader_1x09_P2.54mm_Vertical" (id 2) (at 119.38 39.37 0)
+      (effects (font (size 1.27 1.27)) hide)
+    )
+    (property "Datasheet" "~" (id 3) (at 119.38 39.37 0)
+      (effects (font (size 1.27 1.27)) hide)
+    )
+    (pin "1")
+    (pin "2")
+    (pin "3")
+    (pin "4")
+    (pin "5")
+    (pin "6")
+    (pin "7")
+    (pin "8")
+    (pin "9")
+  )
   (symbol (lib_id "Connector:Conn_01x09_Female") (at 109.22 74.93 0) (mirror y) (unit 1)
     (in_bom yes) (on_board yes) (fields_autoplaced)
@@
       (reference "J24") (unit 1) (value "XT90PW-M") (footprint "SEB:AMASS_XT90PW-M")
     )
-  )
+    (path "/7cb08a70-3f5d-4341-bf6e-21e9f86adbaa"
+      (reference "J25") (unit 1) (value "Conn_01x09_Female") (footprint "Connector_PinHeader_2.54mm:PinHeader_1x09_P2.54mm_Vertical")
+    )
+    (path "/0abad01c-8cfb-4cd7-9f2d-5ad9e9479b46"
+      (reference "J26") (unit 1) (value "Conn_01x09_Female") (footprint "Connector_PinHeader_2.54mm:PinHeader_1x09_P2.54mm_Vertical")
+    )
+    (path "/60bd821a-acde-486a-b846-b5d1e7ebe8d4"
+      (reference "J27") (unit 1) (value "Conn_01x09_Female") (footprint "Connector_PinHeader_2.54mm:PinHeader_1x09_P2.54mm_Vertical")
+    )
+    (path "/4b9e5b04-411b-4437-a64b-0cc9fd79dccd"
+      (reference "J28") (unit 1) (value "Conn_01x09_Female") (footprint "Connector_PinHeader_2.54mm:PinHeader_1x09_P2.54mm_Vertical")
+    )
+  )
