File: ACTIVE_BALANCER/electronique/active_balancer_v1/active_balancer_v1.kicad_sch (KiCad schematic)
At the start: 1 part, among them U1 LTC3300ILXE-2_PBF

Commit message: finished the schematic need a review to make shure everything is okay and after pcb placing & routing while be made. Note this active balancer is for 6s scallable easly for 64s
Parts:
- added C1, C11, C14, C17, C5, C8: ${CBYPASS}, Capacitor_SMD:CP_Elec_8x10, symbol Device:C_Polarized
- added C10, C12, C13, C15, C16, C18, C19, C2, C3, C6, C7, C9: ${CSNUB}, Capacitor_SMD:C_0603_1608Metric_Pad1.08x0.95mm_HandSolder, symbol Device:C
- added C20: ${CBOOST+}, Capacitor_SMD:C_0603_1608Metric_Pad1.08x0.95mm_HandSolder, symbol Device:C
- added C4: ${CBOOST}, Capacitor_SMD:C_0603_1608Metric_Pad1.08x0.95mm_HandSolder, symbol Device:C
- added D1: D_Schottky, Diode_SMD:D_0603_1608Metric_Pad1.05x0.95mm_HandSolder, symbol Device:D_Schottky
- added J1: JST_XH_6S, Connector_JST:JST_XH_B7B-XH-AM_1x07_P2.50mm_Vertical, symbol Connector:Conn_01x07_Socket
- added J2: JST_XH_6pin_SPI, Connector_JST:JST_XH_B6B-XH-AM_1x06_P2.50mm_Vertical, symbol Connector:Conn_01x06_Socket
- added JP1: JUMPER_A1, Jumper:SolderJumper-3_P1.3mm_Open_RoundedPad1.0x1.5mm, symbol Jumper:SolderJumper_3_Open
- added JP2: JUMPER_A2, Jumper:SolderJumper-3_P1.3mm_Open_RoundedPad1.0x1.5mm, symbol Jumper:SolderJumper_3_Open
- added JP3: JUMPER_A3, Jumper:SolderJumper-3_P1.3mm_Open_RoundedPad1.0x1.5mm, symbol Jumper:SolderJumper_3_Open
- added JP4: JUMPER_A4, Jumper:SolderJumper-3_P1.3mm_Open_RoundedPad1.0x1.5mm, symbol Jumper:SolderJumper_3_Open
- added JP5: JUMPER_A5, Jumper:SolderJumper-3_P1.3mm_Open_RoundedPad1.0x1.5mm, symbol Jumper:SolderJumper_3_Open
- added JP6: JUMPER_EN_NUM_ISO_IN, Jumper:SolderJumper-3_P1.3mm_Open_RoundedPad1.0x1.5mm, symbol Jumper:SolderJumper_3_Open
- added JP7: JUMPER_EN_NUM_ISO_OUT, Jumper:SolderJumper-3_P1.3mm_Open_RoundedPad1.0x1.5mm, symbol Jumper:SolderJumper_3_Open
- added JP8: Whatchdog Timer, Jumper:SolderJumper-3_P1.3mm_Open_RoundedPad1.0x1.5mm, symbol Jumper:SolderJumper_3_Open
- added Q1, Q10, Q11, Q12, Q2, Q3, Q4, Q5, Q6, Q7, Q8, Q9: ${FET-N}, active_balancer:SIR882DP_PowerPAK_SO-8_Single, symbol Device:Q_NMOS_Depletion_DGS
- added R1, R10, R14, R18, R22, R26: ${RSENSS}, Resistor_SMD:R_0603_1608Metric_Pad0.98x0.95mm_HandSolder, symbol Device:R
- added R11, R13, R15, R17, R19, R21, R23, R25, R3, R4, R7, R9: ${RSNUB}, Resistor_SMD:R_0603_1608Metric_Pad0.98x0.95mm_HandSolder, symbol Device:R
- added R12, R16, R2, R20, R24, R8: ${RSENSP}, Resistor_SMD:R_0603_1608Metric_Pad0.98x0.95mm_HandSolder, symbol Device:R
- added R27: ${RBOOST+}, Resistor_SMD:R_0603_1608Metric_Pad0.98x0.95mm_HandSolder, symbol Device:R
- added R28: ${RWDT}, Resistor_SMD:R_0603_1608Metric_Pad0.98x0.95mm_HandSolder, symbol Device:R
- added R5: ${RTONP}, Resistor_SMD:R_0603_1608Metric_Pad0.98x0.95mm_HandSolder, symbol Device:R
- added R6: ${RTONS}, Resistor_SMD:R_0603_1608Metric_Pad0.98x0.95mm_HandSolder, symbol Device:R
- added T1, T2, T3, T4, T5, T6: ${TRANSFORMER}, active_balancer:WE-FLYLT_EP13_2381, symbol Device:Transformer_1P_1S
- added U2: ADuM1401xRW, Package_SO:SOIC-16W_7.5x10.3mm_P1.27mm, symbol Isolator:ADuM1401xRW
Connections:
- net LT3300_G6S: now reaches U1.1 (G6S)
- net LT3300_G6S: now also Q12.2 (G)
- net LT3300_I2S: now reaches U1.10 (I2S)
- net LT3300_I2S: now also Q4.3 (S), R10.1
- net LT3300_G1S: now reaches U1.11 (G1S)
- net LT3300_G1S: now also Q2.2 (G)
- net LT3300_I1S: now reaches U1.12 (I1S)
- net LT3300_I1S: now also Q2.3 (S), R1.1
- net LT3300_RTONS: now reaches U1.13 (RTONS)
- net LT3300_RTONS: now also R6.1
- net LT3300_RTONP: now reaches U1.14 (RTONP)
- net LT3300_RTONP: now also R5.1
- net CELL_1-: now reaches U1.15 (CTRL)
- net CELL_1-: now also U1.21 (V-), U1.49 (V-), C1.2, C4.2, J1.7 (Pin_7), JP1.1 (A), JP2.1 (A), JP3.1 (A), JP4.1 (A), JP5.1 (A), JP6.3 (B), JP8.1 (A), R1.2, R10.2, R14.2, R18.2, R2.2, R22.2, R26.2, R5.2, R6.2, U2.15 (GND2), U2.9 (GND2)
- net LT3300_CSBI: now reaches U1.16 (~{CSBI})
- net LT3300_CSBI: now also U2.14 (VOA)
- net LT3300_SCKI: now reaches U1.17 (SCKI)
- net LT3300_SCKI: now also U2.13 (VOB)
- net LT3300_SDI: now reaches U1.18 (SDI)
- net LT3300_SDI: now also J2.3 (Pin_3), U2.12 (VOC), U2.5 (VIC)
- net LT3300_SDO: now reaches U1.19 (SDO)
- net LT3300_SDO: now also J2.2 (Pin_2), U2.11 (VID), U2.6 (VOD)
- net LT3300_I6S: now reaches U1.2 (I6S)
- net LT3300_I6S: now also Q12.3 (S), R26.1
- net LT3300_WDT: now reaches U1.20 (WDT)
- net LT3300_WDT: now also JP8.2 (C)
- net LT3300_I1P: now reaches U1.22 (I1P)
- net LT3300_I1P: now also Q1.3 (S), R2.1
- net LT3300_G1P: now reaches U1.23 (G1P)
- net LT3300_G1P: now also Q1.2 (G)
- net CELL_1+: now reaches U1.24 (C1)
- net CELL_1+: now also C1.1, C5.2, J1.6 (Pin_6), R3.1, R8.2, T1.1 (AA)
- net LT3300_I2P: now reaches U1.25 (I2P)
- net LT3300_I2P: now also Q3.3 (S), R8.1
- net LT3300_G2P: now reaches U1.26 (G2P)
- net LT3300_G2P: now also Q3.2 (G)
- net CELL_2+: now reaches U1.27 (C2)
- net CELL_2+: now also C5.1, C8.2, J1.5 (Pin_5), R12.2, R7.1, T2.1 (AA)
- net LT3300_I3P: now reaches U1.28 (I3P)
- net LT3300_I3P: now also Q5.3 (S), R12.1
- net LT3300_G3P: now reaches U1.29 (G3P)
- net LT3300_G3P: now also Q5.2 (G)
- net LT3300_G5S: now reaches U1.3 (G5S)
- net LT3300_G5S: now also Q10.2 (G)
- net CELL_3+: now reaches U1.30 (C3)
- net CELL_3+: now also C11.2, C8.1, J1.4 (Pin_4), R11.1, R16.2, T3.1 (AA)
- net LT3300_I4P: now reaches U1.31 (I4P)
- net LT3300_I4P: now also Q7.3 (S), R16.1
- net LT3300_G4P: now reaches U1.32 (G4P)
- net LT3300_G4P: now also Q7.2 (G)
- net CELL_4+: now reaches U1.33 (C4)
- net CELL_4+: now also C11.1, C14.2, J1.3 (Pin_3), R15.1, R20.2, T4.1 (AA)
- net LT3300_I5P: now reaches U1.34 (I5P)
- net LT3300_I5P: now also Q9.3 (S), R20.1
- net LT3300_G5P: now reaches U1.35 (G5P)
- net LT3300_G5P: now also Q9.2 (G)
- net CELL_5+: now reaches U1.36 (C5)
- net CELL_5+: now also C14.1, C17.2, J1.2 (Pin_2), R19.1, R24.2, T5.1 (AA)
- net LT3300_I6P: now reaches U1.37 (I6P)
- net LT3300_I6P: now also Q11.3 (S), R24.1
- net LT3300_G6P: now reaches U1.38 (G6P)
- net LT3300_G6P: now also Q11.2 (G)
- net CELL_6+: now reaches U1.39 (C6)
- net CELL_6+: now also C17.1, D1.2 (A), J1.1 (Pin_1), R23.1, T6.1 (AA)
- net LT3300_I5S: now reaches U1.4 (I5S)
- net LT3300_I5S: now also Q10.3 (S), R22.1
- net LT3300_BOOSTP: now reaches U1.40 (BOOSTP)
- net LT3300_BOOSTP: now also C20.1, R27.1
- net LT3300_BOOSTN: now reaches U1.41 (BOOSTN)
- net LT3300_BOOSTN: now also C20.2
- net LT3300_BOOST: now reaches U1.42 (BOOST)
- net LT3300_BOOST: now also U1.48 (VREG), C4.1, JP1.3 (B), JP2.3 (B), JP3.3 (B), JP4.3 (B), JP5.3 (B), JP6.1 (A), R28.1, U2.16 (VDD2)
- net LT3300_A0: now reaches U1.43 (A0)
- net LT3300_A0: now also JP1.2 (C)
- net LT3300_A1: now reaches U1.44 (A1)
- net LT3300_A1: now also JP2.2 (C)
- net LT3300_A2: now reaches U1.45 (A2)
- net LT3300_A2: now also JP3.2 (C)
- net LT3300_A3: now reaches U1.46 (A3)
- net LT3300_A3: now also JP4.2 (C)
- net LT3300_A4: now reaches U1.47 (A4)
- net LT3300_A4: now also JP5.2 (C)
- net LT3300_G4S: now reaches U1.5 (G4S)
- net LT3300_G4S: now also Q8.2 (G)
- net LT3300_I4S: now reaches U1.6 (I4S)
- net LT3300_I4S: now also Q8.3 (S), R18.1
- net LT3300_G3S: now reaches U1.7 (G3S)
- net LT3300_G3S: now also Q6.2 (G)
- net LT3300_I3S: now reaches U1.8 (I3S)
- net LT3300_I3S: now also Q6.3 (S), R14.1
- net LT3300_G2S: now reaches U1.9 (G2S)
- net LT3300_G2S: now also Q4.2 (G)
- new net: D1.1 (K), R27.2
- new net: C12.1, R15.2
- new net: C12.2, Q7.1 (D), T4.2 (AB)
- new net: JP8.3 (B), R28.2
- new net: R4.1, T1.4 (SB)
- new net: C3.1, R4.2
- new net: C18.2, Q11.1 (D), T6.2 (AB)
- new net: C13.1, R17.2
- new net: C13.2, Q8.1 (D), T4.3 (SA)
- new net: C6.2, Q3.1 (D), T2.2 (AB)
- new net: C7.2, Q4.1 (D), T2.3 (SA)
- new net: R9.1, T2.4 (SB)
- new net: C3.2, Q2.1 (D), T1.3 (SA)
- new net: C2.2, Q1.1 (D), T1.2 (AB)
- new net: C6.1, R7.2
- new net: C9.2, Q5.1 (D), T3.2 (AB)
- new net: C10.2, Q6.1 (D), T3.3 (SA)
- new net: R13.1, T3.4 (SB)
- new net: R21.1, T5.4 (SB)
- new net: C16.1, R21.2
- new net: C10.1, R13.2
- new net: C18.1, R23.2
- new net: JP6.2 (C), U2.10 (VE2)
- new net: C7.1, R9.2
- new net: C9.1, R11.2
- new net: R25.1, T6.4 (SB)
- new net: C19.1, R25.2
- new net: C2.1, R3.2
- new net: R17.1, T4.4 (SB)
- new net: C15.1, R19.2
- new net: C15.2, Q9.1 (D), T5.2 (AB)
- new net: C16.2, Q10.1 (D), T5.3 (SA)
- new net: C19.2, Q12.1 (D), T6.3 (SA)
- new net: JP7.2 (C), U2.7 (VE1)
- new net 5V: J2.6 (Pin_6), JP7.1 (A), U2.1 (VDD1)
- new net GND: J2.1 (Pin_1), JP7.3 (B), U2.2 (GND1), U2.8 (GND1)
- new net LT3300_CS: J2.5 (Pin_5), U2.3 (VIA)
- new net LT3300_SCK: J2.4 (Pin_4), U2.4 (VIB)
Other:
- note added: "Active Balance Stage 6S"
- note added: "Always connect a minimum of 3 cells If connecte less than 6 cells always connect the highest cell in the pack to the cell 6 and short the other unused pin together -> see doc page 32 for more info"
- note added: "Battery connector"
- note added: "LTC3300-2"
- note added: "Linear Voltage Regulator Output & CTRL pin setup"
- note added: "Not sure of the RWDT value to try? Whatchdog cutoff the balancing process if no communication on spi is detected for more than 1.5s Pull high to enable Pull low to disable"
- note added: "SPI Address & Configuration"
- note added: "SPI Communication & Isolation"
- note added: "SPI connector"
- note added: "The ctrl pin is pulled low because we use the multiple transformer configuration"
- note added: "The spi line for all LTC3300-2 are in parallel and each IC have a unique id that we put in the begining of each command"
- note added: "Watchdog safety"
- company: (none) -> VOLTN SOLEX
- title: (none) -> 6S Active Balancer
- moved on the sheet: U1

Commit message: Updated the pcb rooting and created a step file to check the finting in fusion 360
Parts:
- removed J1: JST_XH_6S, Connector_JST:JST_XH_B7B-XH-AM_1x07_P2.50mm_Vertical, symbol Connector:Conn_01x07_Socket
- added C21, C22, C23, C24, C25, C26: ${CBYPASS_DECOP}, Capacitor_SMD:C_0603_1608Metric_Pad1.08x0.95mm_HandSolder, symbol Device:C
- added J1, J10, J3, J4, J5, J6, J7, J8, J9: Conn_01x01_Socket, Connector_PinSocket_2.54mm:PinSocket_1x01_P2.54mm_Vertical, symbol Connector:Conn_01x01_Socket
Connections:
- net CELL_1+: now also C25.2, C26.1, J1.1 (Pin_1)
- net CELL_1-: now also C26.2, J3.1 (Pin_1), J9.1 (Pin_1)
- net CELL_2+: now also C24.2, C25.1, J4.1 (Pin_1)
- net CELL_3+: now also C23.2, C24.1, J5.1 (Pin_1)
- net CELL_4+: now also C22.2, C23.1, J6.1 (Pin_1)
- net CELL_5+: now also C21.2, C22.1, J7.1 (Pin_1)
- net CELL_6+: now also C21.1, J10.1 (Pin_1), J8.1 (Pin_1)
- net LT3300_SDI: no longer J2.3 (Pin_3), U2.5 (VIC)
- net LT3300_SDO: no longer J2.2 (Pin_2), U2.6 (VOD)
- net LT3300_CS renamed GLOBAL_LT3300_CS
- net LT3300_SCK renamed GLOBAL_LT3300_SCK
- new net GLOBAL_LT3300_SDI: J2.3 (Pin_3), U2.5 (VIC)
- new net GLOBAL_LT3300_SDO: J2.2 (Pin_2), U2.6 (VOD)
